File: Can3DPrinter4Motor.kicad_pcb (KiCad board)
At the start: 6 copper layers, 0 parts

Commit message: Complete schematics Assign every value (very few exceptions) Change TCM5160 from on-board to separate module Add fuses Add power supplies (LDO + 2x buck converter)
Parts:
- added C201: 14pF, Capacitor_SMD:C_0402_1005Metric, F.Cu at (62.0, 126.0)
- added C202: 14pF, Capacitor_SMD:C_0402_1005Metric, F.Cu at (65.0, 126.0)
- added C211: 100nF, Capacitor_SMD:C_0402_1005Metric, F.Cu at (69.6, 112.5)
- added C221: 1uF, Capacitor_SMD:C_0402_1005Metric, F.Cu at (65.8, 111.0)
- added C222: 1uF, Capacitor_SMD:C_0402_1005Metric, F.Cu at (66.8, 111.0)
- added C231: 100nF, Capacitor_SMD:C_0402_1005Metric, F.Cu at (65.5, 122.4)
- added C232: 100nF, Capacitor_SMD:C_0402_1005Metric, F.Cu at (63.8, 111.0)
- added C233: 100nF, Capacitor_SMD:C_0402_1005Metric, F.Cu at (69.6, 113.5)
- added C234: 100nF, Capacitor_SMD:C_0402_1005Metric, F.Cu at (67.8, 111.0)
- added C235: 100nF, Capacitor_SMD:C_0402_1005Metric, F.Cu at (69.6, 117.6)
- added C236: 100nF, Capacitor_SMD:C_0402_1005Metric, F.Cu at (64.8, 111.0)
- added C237: 100nF, Capacitor_SMD:C_0402_1005Metric, F.Cu at (58.9, 113.5)
- added C238: 100nF, Capacitor_SMD:C_0402_1005Metric, F.Cu at (64.5, 122.4)
- added C239: 100nF, Capacitor_SMD:C_0402_1005Metric, F.Cu at (58.7, 117.6)
- added C301: 10uF, Capacitor_SMD:C_1206_3216Metric, F.Cu at (156.6, 180.3)
- added C302: 10uF, Capacitor_SMD:C_1206_3216Metric, F.Cu at (156.6, 177.8)
- added C311: 10uF, Capacitor_SMD:C_1206_3216Metric, F.Cu at (132.9, 186.9)
- added C312: 10nF, Capacitor_SMD:C_0603_1608Metric, F.Cu at (129.8, 182.4)
- added C313: 10uF, Capacitor_SMD:C_1206_3216Metric, F.Cu at (122.2, 178.6)
- added C321: 10uF, Capacitor_SMD:C_1206_3216Metric, F.Cu at (94.0, 185.4)
- added C322: 10nF, Capacitor_SMD:C_0603_1608Metric, F.Cu at (88.9, 181.4)
- added C323: 10uF, Capacitor_SMD:C_1206_3216Metric, F.Cu at (83.1, 177.3)
- added C324: 10uF, Capacitor_SMD:C_1206_3216Metric, F.Cu at (83.1, 179.8)
- added C601: 470nF, Capacitor_SMD:C_0603_1608Metric, F.Cu at (313.7, 34.0)
- added C611: 100nF, Capacitor_SMD:C_0402_1005Metric, F.Cu at (322.8, 13.2)
- added C612: 100nF, Capacitor_SMD:C_0402_1005Metric, F.Cu at (334.0, 13.2)
- added C701: 470nF, Capacitor_SMD:C_0603_1608Metric, F.Cu at (315.2, 77.0)
- added C711: 100nF, Capacitor_SMD:C_0402_1005Metric, F.Cu at (322.1, 57.6)
- added C712: 100nF, Capacitor_SMD:C_0402_1005Metric, F.Cu at (333.2, 57.6)
- added C801: 470nF, Capacitor_SMD:C_0603_1608Metric, F.Cu at (314.5, 123.7)
- added C811: 100nF, Capacitor_SMD:C_0402_1005Metric, F.Cu at (322.1, 105.6)
- added C812: 100nF, Capacitor_SMD:C_0402_1005Metric, F.Cu at (333.2, 105.6)
- added C901: 470nF, Capacitor_SMD:C_0603_1608Metric, F.Cu at (315.5, 170.9)
- added C911: 100nF, Capacitor_SMD:C_0402_1005Metric, F.Cu at (323.6, 152.1)
- added C912: 100nF, Capacitor_SMD:C_0402_1005Metric, F.Cu at (334.8, 152.1)
- added D101: White, LED_SMD:LED_0402_1005Metric, F.Cu at (19.2, 39.4)
- added D102: White, LED_SMD:LED_0402_1005Metric, F.Cu at (19.2, 40.9)
- added D103: White, LED_SMD:LED_0402_1005Metric, F.Cu at (19.2, 42.4)
- added D104: White, LED_SMD:LED_0402_1005Metric, F.Cu at (19.2, 43.9)
- added D105: White, LED_SMD:LED_0402_1005Metric, F.Cu at (19.2, 45.5)
- added D301: D_Schottky, Diode_SMD:D_SMA, F.Cu at (160.3, 186.2)
- added D311: B5819W, Diode_SMD:D_SOD-123, F.Cu at (132.3, 179.1)
- added D321: B5819W, Diode_SMD:D_SOD-123, F.Cu at (93.5, 177.3)
- added D601: White, LED_SMD:LED_0402_1005Metric, F.Cu at (329.4, 26.2)
- added D701: White, LED_SMD:LED_0402_1005Metric, F.Cu at (328.9, 71.4)
- added D801: White, LED_SMD:LED_0402_1005Metric, F.Cu at (330.7, 113.8)
- added D901: White, LED_SMD:LED_0402_1005Metric, F.Cu at (330.9, 161.0)
- added F101: 65V 20A, Custom:Fuse_2410_6125Metric, F.Cu at (57.8, 44.7)
- added F102: 65V 20A, Custom:Fuse_2410_6125Metric, F.Cu at (57.8, 37.1)
- added F103: 65V 20A, Custom:Fuse_2410_6125Metric, F.Cu at (57.8, 40.9)
- added F401: 250mA, Resistor_SMD:R_0603_1608Metric, F.Cu at (-28.4, 93.5)
- added F402: 250mA, Resistor_SMD:R_0603_1608Metric, F.Cu at (-28.4, 101.1)
- added F403: 250mA, Resistor_SMD:R_0603_1608Metric, F.Cu at (-28.4, 108.7)
- added F404: 250mA, Resistor_SMD:R_0603_1608Metric, F.Cu at (-28.4, 116.3)
- added H101: MountingHole_Pad, MountingHole:MountingHole_2.2mm_M2_ISO7380_Pad, F.Cu at (15.5, 15.2)
- added H102: MountingHole_Pad, MountingHole:MountingHole_2.2mm_M2_ISO7380_Pad, F.Cu at (282.4, 14.7)
- added H103: MountingHole_Pad, MountingHole:MountingHole_2.2mm_M2_ISO7380_Pad, F.Cu at (278.6, 160.3)
- added H104: MountingHole_Pad, MountingHole:MountingHole_2.2mm_M2_ISO7380_Pad, F.Cu at (17.8, 193.0)
- added H111: MountingHole_Pad, Custom:Tooling Hole (JLCPCB), F.Cu at (15.7, 21.3)
- added H112: MountingHole_Pad, Custom:Tooling Hole (JLCPCB), F.Cu at (15.7, 24.4)
- added J101: Molex Micro-Fit 3.0 2x03 - CAN bus, Connector_Molex:Molex_Micro-Fit_3.0_43045-0612_2x03_P3.00mm_Vertical, F.Cu at (72.3, 39.3)
- added J102: Molex Micro-Fit 3.0 2x03 - CAN bus, Connector_Molex:Molex_Micro-Fit_3.0_43045-0612_2x03_P3.00mm_Vertical, F.Cu at (72.3, 49.3)
- added J111: RGB, Connector_JST:JST_XH_B3B-XH-A_1x03_P2.50mm_Vertical, F.Cu at (-21.6, 12.9)
- added J121: Temperature, Connector_JST:JST_XH_B2B-XH-A_1x02_P2.50mm_Vertical, F.Cu at (-68.6, 11.6)
- added J122: Temperature, Connector_JST:JST_XH_B2B-XH-A_1x02_P2.50mm_Vertical, F.Cu at (-68.6, 19.4)
- added J123: Temperature, Connector_JST:JST_XH_B2B-XH-A_1x02_P2.50mm_Vertical, F.Cu at (-68.6, 27.2)
- added J124: Temperature, Connector_JST:JST_XH_B2B-XH-A_1x02_P2.50mm_Vertical, F.Cu at (-68.6, 35.0)
- added J131: Heating Enable, Connector_JST:JST_XH_B2B-XH-A_1x02_P2.50mm_Vertical, F.Cu at (-70.8, 66.4)
- added J132: Heating Enable, Connector_JST:JST_XH_B2B-XH-A_1x02_P2.50mm_Vertical, F.Cu at (-70.8, 74.2)
- added J141: Limit Switch, Connector_JST:JST_XH_B3B-XH-A_1x03_P2.50mm_Vertical, F.Cu at (-34.5, 36.8)
- added J142: Limit Switch, Connector_JST:JST_XH_B3B-XH-A_1x03_P2.50mm_Vertical, F.Cu at (-34.5, 44.6)
- added J143: Limit Switch, Connector_JST:JST_XH_B3B-XH-A_1x03_P2.50mm_Vertical, F.Cu at (-34.5, 52.4)
- added J144: Limit Switch, Connector_JST:JST_XH_B3B-XH-A_1x03_P2.50mm_Vertical, F.Cu at (-34.5, 60.2)
- added J301: USB_C_Receptacle_USB2.0, Connector_USB:USB_C_Receptacle_GCT_USB4105-xx-A_16P_TopMnt_Horizontal, F.Cu at (56.6, 151.1)
- added J401: Fan Connector, Connector_JST:JST_XH_B2B-XH-A_1x02_P2.50mm_Vertical, F.Cu at (-23.3, 90.9)
- added J402: Fan Voltage Selection, Connector_PinHeader_2.54mm:PinHeader_2x03_P2.54mm_Vertical, F.Cu at (-16.0, 88.9)
- added J403: Fan Connector, Connector_JST:JST_XH_B2B-XH-A_1x02_P2.50mm_Vertical, F.Cu at (-23.3, 98.5)
- added J404: Fan Voltage Selection, Connector_PinHeader_2.54mm:PinHeader_2x03_P2.54mm_Vertical, F.Cu at (-16.0, 96.5)
- added J405: Fan Connector, Connector_JST:JST_XH_B2B-XH-A_1x02_P2.50mm_Vertical, F.Cu at (-23.3, 106.2)
- added J406: Fan Voltage Selection, Connector_PinHeader_2.54mm:PinHeader_2x03_P2.54mm_Vertical, F.Cu at (-16.0, 104.1)
- added J407: Fan Connector, Connector_JST:JST_XH_B2B-XH-A_1x02_P2.50mm_Vertical, F.Cu at (-23.3, 113.8)
- added J408: Fan Voltage Selection, Connector_PinHeader_2.54mm:PinHeader_2x03_P2.54mm_Vertical, F.Cu at (-16.0, 111.8)
- added J601: Motor Connector, Connector_JST:JST_XH_B4B-XH-A_1x04_P2.50mm_Vertical, F.Cu at (321.3, 22.7)
- added J602: Encoder, Connector_JST:JST_XH_B5B-XH-A_1x05_P2.50mm_Vertical, F.Cu at (314.6, 13.2)
- added J603: Direction, Connector_PinHeader_2.54mm:PinHeader_2x02_P2.54mm_Vertical, F.Cu at (327.1, 10.4)
- added J701: Motor Connector, Connector_JST:JST_XH_B4B-XH-A_1x04_P2.50mm_Vertical, F.Cu at (322.9, 65.6)
- added J702: Encoder, Connector_JST:JST_XH_B5B-XH-A_1x05_P2.50mm_Vertical, F.Cu at (316.1, 56.2)
- added J703: Direction, Connector_PinHeader_2.54mm:PinHeader_2x02_P2.54mm_Vertical, F.Cu at (326.4, 54.9)
- added J801: Motor Connector, Connector_JST:JST_XH_B4B-XH-A_1x04_P2.50mm_Vertical, F.Cu at (322.1, 112.3)
- added J802: Encoder, Connector_JST:JST_XH_B5B-XH-A_1x05_P2.50mm_Vertical, F.Cu at (315.4, 102.9)
- added J803: Direction, Connector_PinHeader_2.54mm:PinHeader_2x02_P2.54mm_Vertical, F.Cu at (326.4, 102.9)
- added J901: Motor Connector, Connector_JST:JST_XH_B4B-XH-A_1x04_P2.50mm_Vertical, F.Cu at (323.1, 159.6)
- added J902: Encoder, Connector_JST:JST_XH_B5B-XH-A_1x05_P2.50mm_Vertical, F.Cu at (316.4, 150.1)
- added J903: Direction, Connector_PinHeader_2.54mm:PinHeader_2x02_P2.54mm_Vertical, F.Cu at (327.9, 149.3)
- added L311: 10uH, Inductor_SMD:L_Sunlord_MWSA0503S, F.Cu at (127.8, 178.6)
- added L321: 10uH, Inductor_SMD:L_Sunlord_MWSA0503S, F.Cu at (88.9, 177.3)
- added Q301: Si2309CDS, Package_TO_SOT_SMD:SOT-23, F.Cu at (156.5, 186.2)
- added Q401: BSS138, Package_TO_SOT_SMD:SOT-23, F.Cu at (-28.4, 90.9)
- added Q402: BSS138, Package_TO_SOT_SMD:SOT-23, F.Cu at (-28.4, 98.6)
- added Q403: BSS138, Package_TO_SOT_SMD:SOT-23, F.Cu at (-28.4, 106.2)
- added Q404: BSS138, Package_TO_SOT_SMD:SOT-23, F.Cu at (-28.4, 113.8)
- added R101: 90k, Resistor_SMD:R_0603_1608Metric, F.Cu at (21.8, 39.4)
- added R102: 42k, Resistor_SMD:R_0603_1608Metric, F.Cu at (21.8, 40.9)
- added R103: 18k, Resistor_SMD:R_0603_1608Metric, F.Cu at (21.8, 42.4)
- added R104: 4.7k, Resistor_SMD:R_0603_1608Metric, F.Cu at (21.8, 43.9)
- added R105: 600, Resistor_SMD:R_0603_1608Metric, F.Cu at (21.8, 45.5)
- added R201: 1k, Resistor_SMD:R_0402_1005Metric, F.Cu at (63.5, 125.5)
- added R211: 27.4R, Resistor_SMD:R_0402_1005Metric, F.Cu at (55.9, 140.2)
- added R212: 27.4R, Resistor_SMD:R_0402_1005Metric, F.Cu at (56.9, 140.2)
- added R221: 10k, Resistor_SMD:R_0603_1608Metric, F.Cu at (55.6, 101.6)
- added R301: 10k, Resistor_SMD:R_0603_1608Metric, F.Cu at (157.0, 188.7)
- added R311: 10k, Resistor_SMD:R_0603_1608Metric, F.Cu at (122.7, 184.2)
- added R312: 3.2k, Resistor_SMD:R_0603_1608Metric, F.Cu at (122.7, 187.2)
- added R321: 100k, Resistor_SMD:R_0603_1608Metric, F.Cu at (92.0, 184.7)
- added R322: 47k, Resistor_SMD:R_0603_1608Metric, F.Cu at (84.6, 182.6)
- added R323: 3.4k, Resistor_SMD:R_0603_1608Metric, F.Cu at (84.6, 185.7)
- added R331: 5.1k, Resistor_SMD:R_0603_1608Metric, F.Cu at (55.1, 144.7)
- added R332: 5.1k, Resistor_SMD:R_0603_1608Metric, F.Cu at (58.2, 144.7)
- added R501: 10k, Resistor_SMD:R_0603_1608Metric, F.Cu at (292.3, 91.4)
- added R601: 47k, Resistor_SMD:R_0603_1608Metric, F.Cu at (332.0, 24.6)
- added R602: 4.7k, Resistor_SMD:R_0603_1608Metric, F.Cu at (332.0, 26.2)
- added R611: 10k, Resistor_SMD:R_0603_1608Metric, F.Cu at (324.6, 13.8)
- added R612: 47k, Resistor_SMD:R_0603_1608Metric, F.Cu at (323.8, 11.4)
- added R613: 10k, Resistor_SMD:R_0603_1608Metric, F.Cu at (332.2, 13.8)
- added R614: 47k, Resistor_SMD:R_0603_1608Metric, F.Cu at (333.1, 11.4)
- added R701: 47k, Resistor_SMD:R_0603_1608Metric, F.Cu at (331.5, 69.8)
- added R702: 4.7k, Resistor_SMD:R_0603_1608Metric, F.Cu at (331.5, 71.4)
- added R711: 10k, Resistor_SMD:R_0603_1608Metric, F.Cu at (323.9, 58.2)
- added R712: 47k, Resistor_SMD:R_0603_1608Metric, F.Cu at (323.0, 55.9)
- added R713: 10k, Resistor_SMD:R_0603_1608Metric, F.Cu at (331.5, 58.2)
- added R714: 47k, Resistor_SMD:R_0603_1608Metric, F.Cu at (332.3, 55.9)
- added R801: 47k, Resistor_SMD:R_0603_1608Metric, F.Cu at (333.2, 112.3)
- added R802: 4.7k, Resistor_SMD:R_0603_1608Metric, F.Cu at (333.2, 113.8)
- added R811: 10k, Resistor_SMD:R_0603_1608Metric, F.Cu at (323.9, 106.2)
- added R812: 47k, Resistor_SMD:R_0603_1608Metric, F.Cu at (323.0, 103.9)
- added R813: 10k, Resistor_SMD:R_0603_1608Metric, F.Cu at (331.5, 106.2)
- added R814: 47k, Resistor_SMD:R_0603_1608Metric, F.Cu at (332.3, 103.9)
- added R901: 47k, Resistor_SMD:R_0603_1608Metric, F.Cu at (333.5, 159.5)
- added R902: 4.7k, Resistor_SMD:R_0603_1608Metric, F.Cu at (333.5, 161.0)
- added R911: 10k, Resistor_SMD:R_0603_1608Metric, F.Cu at (325.4, 152.7)
- added R912: 47k, Resistor_SMD:R_0603_1608Metric, F.Cu at (324.5, 150.4)
- added R913: 10k, Resistor_SMD:R_0603_1608Metric, F.Cu at (333.0, 152.7)
- added R914: 47k, Resistor_SMD:R_0603_1608Metric, F.Cu at (333.8, 150.4)
- added TP101: TestPoint, TestPoint:TestPoint_Pad_D1.0mm, F.Cu at (22.6, 14.5)
- added TP102: TestPoint, TestPoint:TestPoint_Pad_D1.0mm, F.Cu at (22.6, 16.8)
- added TP103: TestPoint, TestPoint:TestPoint_Pad_D1.0mm, F.Cu at (22.6, 21.3)
- added TP104: TestPoint, TestPoint:TestPoint_Pad_D1.0mm, F.Cu at (22.6, 23.6)
- added TP105: TestPoint, TestPoint:TestPoint_Pad_D1.0mm, F.Cu at (22.6, 25.9)
- added TP106: TestPoint, TestPoint:TestPoint_Pad_D1.0mm, F.Cu at (22.6, 28.2)
- added TP107: TestPoint, TestPoint:TestPoint_Pad_D1.0mm, F.Cu at (22.6, 19.1)
- added U201: RP2040, Package_DFN_QFN:QFN-56-1EP_7x7mm_P0.4mm_EP3.2x3.2mm, F.Cu at (64.1, 116.6)
- added U202: W25Q128JVS, Package_SO:SOIC-8_5.23x5.23mm_P1.27mm, F.Cu at (55.6, 105.7)
- added U301: AMS1117-3.3, Package_TO_SOT_SMD:SOT-223-3_TabPin2, F.Cu at (163.4, 177.8)
- added U311: TPS5430DDA, Package_SO:TI_SO-PowerPAD-8_ThermalVias, F.Cu at (127.8, 185.9)
- added U321: MP2359DJ, Package_TO_SOT_SMD:SOT-23-6, F.Cu at (88.9, 183.9)
- added U601: FYSETC TMC5160, Custom:FYSETC TMC5160, F.Cu at (303.3, 17.5)
- added U701: FYSETC TMC5160, Custom:FYSETC TMC5160, F.Cu at (304.8, 60.5)
- added U801: FYSETC TMC5160, Custom:FYSETC TMC5160, F.Cu at (304.0, 107.2)
- added U901: FYSETC TMC5160, Custom:FYSETC TMC5160, F.Cu at (305.1, 154.4)
- added Y201: 12MHz, Crystal:Crystal_SMD_5032-4Pin_5.0x3.2mm, F.Cu at (62.7, 128.5)
Routing:
- net /CAN 24V: track 0.00 -> 29.9 mm
- net /CAN 48V: track 0.00 -> 25.1 mm
- net +3V3: track 0.00 -> 24.2 mm
- net /Microcontroller/XIN: track 0.00 -> 10.6 mm
- net +5V: track 0.00 -> 10.5 mm
- net Net-(D321-K): track 0.00 -> 10.3 mm
- net USB D-: track 1.41 -> 11.0 mm
- net +12V: track 0.00 -> 8.67 mm
- net USB D+: track 0.00 -> 8.44 mm
- net Net-(D311-K): track 0.00 -> 8.23 mm
- net +1V1: track 0.00 -> 5.70 mm
- net /Motor Drivers/Motor 4/M4_B2: track 0.00 -> 5.38 mm
- net /Motor Drivers/Motor 4/M4_A2: track 0.00 -> 5.38 mm
- net /Motor Drivers/Motor 3/M3_B2: track 0.00 -> 5.38 mm
- net /Motor Drivers/Motor 3/M3_A2: track 0.00 -> 5.38 mm
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Other:
- board text added: "12V"
- board text added: "1V1"
- board text added: "24V"
- board text added: "3V3"
- board text added: "48V"
- board text added: "48V 24V CAN-H"
- board text added: "5V"
- board text added: "5V 12V 24V"
- board text added: "5V A B N/Z GND"
- board text added: "5V RGB GND"
- board text added: "5V Switch GND"
- board text added: "A2 A1 B1 B2"
- board text added: "GND 5V"
- board text added: "GND GND CAN-L"
- board text added: "GND Switch"
- board text added: "GND Temp"
- board text added: "USB"

Commit message: WIP PCB placement, minor fixes
Parts:
- C601, C701, C801, C901, F401, F402, F403, F404, Q401, Q402, Q403, Q404, R501: moved to B.Cu
- moved J131 290.0 mm to (214.7, 117.3)
- moved J132 289.9 mm to (214.7, 124.2)
- moved J121 279.0 mm to (194.9, 103.6)
- moved J122 278.7 mm to (194.9, 110.5)
- moved J123 278.4 mm to (194.9, 117.3)
- moved J124 278.1 mm to (194.9, 124.2)
- moved J111 253.0 mm to (214.7, 103.6)
- moved J141 247.2 mm to (203.5, 103.6)
- moved J142 247.0 mm to (203.5, 110.5)
- moved J143 246.7 mm to (203.5, 117.3)
- moved J144 246.5 mm to (203.5, 124.2)
- moved R601 195.6 mm to (141.2, 67.8), turned to 90 degrees
- moved C612 194.3 mm to (143.6, 52.1), turned to 0 degrees
- moved R614 193.8 mm to (143.1, 50.0), turned to 90 degrees
- moved R602 193.8 mm to (142.7, 67.8), turned to 90 degrees
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Connections:
- J102 pad 6: unconnected-(J102-Pin_6-Pad6) -> GND
Routing:
- net GND: track 0.00 -> 110.1 mm, vias 0 -> 27
- net +5V: track 10.5 -> 86.2 mm, vias 0 -> 8
- net ~{MOTOR ENABLE}: track 0.00 -> 72.9 mm
- net SPI MOSI: track 0.00 -> 72.0 mm
- net SPI CLK: track 0.00 -> 72.0 mm
- net SPI MISO: track 0.00 -> 72.0 mm
- net M2 REF R: track 0.00 -> 26.5 mm, vias 0 -> 1
- net M4 REF R: track 0.00 -> 26.2 mm, vias 0 -> 1
- net M1 REF R: track 0.00 -> 26.2 mm, vias 0 -> 1
- net M3 REF R: track 0.00 -> 26.2 mm, vias 0 -> 1
- net M4 OUT STEP: track 0.00 -> 26.1 mm
- net M1 OUT STEP: track 0.00 -> 26.0 mm
- net M3 OUT STEP: track 0.00 -> 26.0 mm
- net M2 OUT STEP: track 0.00 -> 26.0 mm
- net M2 REF L: track 0.00 -> 23.3 mm, vias 0 -> 1
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- added copper zone on In3.Cu, net +24V
- added copper zone on In2.Cu, net +5V
- added copper zone on F.Cu, net /Power Supply/VIN
Other:
- board outline added: 142.2 x 88.4 mm
- board text added: "Left Right"
- board text removed: "GND Switch"

Commit message: More PCB placement, fix 48V for Motors
Parts:
- moved H112 206.5 mm to (206.8, 97.0)
- moved H104 125.6 mm to (101.3, 99.3)
- moved H111 94.4 mm to (105.2, 44.6)
- moved H101 90.7 mm to (101.3, 44.5)
- moved H103 83.3 mm to (213.9, 108.0)
- moved H102 76.6 mm to (211.8, 44.5)
- moved R321 70.8 mm to (119.8, 84.5), turned to 180 degrees
- moved D105 70.1 mm to (140.7, 100.1), turned to 90 degrees
- moved D104 69.1 mm to (139.2, 100.1), turned to 90 degrees
- moved U321 69.1 mm to (120.7, 81.4), turned to -90 degrees
- moved C321 68.2 mm to (122.1, 86.7), turned to 0 degrees
- moved D103 68.1 mm to (137.7, 100.1), turned to 90 degrees
- moved R323 68.0 mm to (121.9, 78.6), turned to 0 degrees
- moved D102 67.2 mm to (136.1, 100.1), turned to 90 degrees
- moved R105 67.0 mm to (140.7, 97.5), turned to 90 degrees
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Connections:
- U201 pad 38: unconnected-(U201-GPIO26_ADC0-Pad38) -> Temp 1
- U201 pad 39: unconnected-(U201-GPIO27_ADC1-Pad39) -> Temp 2
- U201 pad 40: unconnected-(U201-GPIO28_ADC2-Pad40) -> Temp 3
- U201 pad 41: unconnected-(U201-GPIO29_ADC3-Pad41) -> Temp 4
- U601 pad 13: +24V -> +48V
- U701 pad 13: +24V -> +48V
- U801 pad 13: +24V -> +48V
- U901 pad 13: +24V -> +48V
Routing:
- net +12V: track 8.48 -> 64.8 mm
- net FAN1: track 0.00 -> 55.3 mm, vias 0 -> 1
- net FAN2: track 0.00 -> 45.0 mm, vias 0 -> 1
- net +24V: track 6.62 -> 49.7 mm
- net FAN3: track 0.00 -> 38.8 mm
- net +3V3: track 23.5 -> 61.8 mm, vias 9 -> 11
- net FAN4: track 0.00 -> 33.0 mm
- net VUSB: track 0.00 -> 22.7 mm, vias 0 -> 3
- net +5V: track 86.2 -> 68.5 mm, vias 8 -> 17
- net unconnected-(J301-SHIELD-PadS1): track 0.00 -> 17.0 mm
- net M4 OUT STEP: track 26.1 -> 14.2 mm, vias 0 -> 1
- net GND: track 110.1 -> 121.6 mm, vias 27 -> 41
- net M1 OUT STEP: track 26.0 -> 17.0 mm, vias 0 -> 1
- net M3 OUT STEP: track 26.0 -> 17.0 mm, vias 0 -> 1
- net M2 OUT STEP: track 26.0 -> 17.0 mm, vias 0 -> 1
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- added copper zone on In2.Cu, net +3V3
- added copper zone on B.Cu, net +48V
- added copper zone on F.Cu, net +48V
- added copper zone on In1.Cu, net +48V
- added copper zone on In2.Cu, net +48V
- added copper zone on In3.Cu, net +48V
- added copper zone on In4.Cu, net +48V
- added copper zone on B.Cu, net +5V
- added copper zone on F.Cu, net +5V
- added copper zone on In1.Cu, net +5V
- added copper zone on In3.Cu, net +5V
- added copper zone on In4.Cu, net +5V
- added copper zone on B.Cu, net /CAN 24V
- added copper zone on F.Cu, net /CAN 24V
- added copper zone on In1.Cu, net /CAN 24V
- added copper zone on In2.Cu, net /CAN 24V
- added copper zone on In3.Cu, net /CAN 24V
- added copper zone on In4.Cu, net /CAN 24V
- removed copper zone on In3.Cu, net +24V
Other:
- board size 142.2 x 88.4 mm -> 115.1 x 59.4 mm
- board text added: "5 A B N -"
- board text added: "5V A B N -"
- board text added: "CAN"
- board text added: "GND"
- board text added: "H"
- board text added: "L"
- board text removed: "48V 24V CAN-H"
- board text removed: "5V A B N/Z GND"
- board text removed: "GND GND CAN-L"
- board text removed: "Left Right"
