File: 4MotorCAN.kicad_pcb (KiCad board)
At the start: 6 copper layers, 115.1 x 59.4 mm, 160 parts, among them J101 Molex Micro-Fit 3.0 2x03 - CA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, J102 Molex Micro-Fit 3.0 2x03 - CA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, J111 RGB, J121 Temperature, J122 Temperature, J123 Temperature, J124 Temperature, J131 Heating Enable, J132 Heating Enable, J141 Limit Switch, J142 Limit Switch, J143 Limit Switch, J144 Limit Switch, J301 USB_C_Receptacle_USB2.0, J401 Fan Connector, J402 Fan Voltage Selection, J403 Fan Connector, J404 Fan Voltage Selection, J405 Fan Connector, J406 Fan Voltage Selection, J407 Fan Connector, J408 Fan Voltage Selection, J601 Motor Connector, J602 Encoder, J603 Direction, J701 Motor Connector, J702 Encoder, J703 Direction, J801 Motor Connector, J802 Encoder, J803 Direction, J901 Motor Connector, J902 Encoder, J903 Direction, Q301 Si2309CDS, Q401 BSS138, Q402 BSS138, Q403 BSS138, Q404 BSS138, U201 RP2040, U202 W25Q128JVS, U301 AMS1117-3.3, U311 TPS5430DDA, U321 MP2359DJ, U601 FYSETC TMC5160, U701 FYSETC TMC5160, U801 FYSETC TMC5160, U901 FYSETC TMC5160, Y201 12MHz

Commit message: Finish wiring PCB
Parts:
- removed TP102, TP103, TP104, TP105, TP106: TestPoint, TestPoint:TestPoint_Pad_D1.0mm
- added C602: ???, Capacitor_THT:CP_Radial_D6.3mm_P2.50mm, F.Cu at (132.5, 55.6)
- added C702: ???, Capacitor_THT:CP_Radial_D6.3mm_P2.50mm, F.Cu at (155.1, 55.6)
- added C802: ???, Capacitor_THT:CP_Radial_D6.3mm_P2.50mm, F.Cu at (177.9, 55.6)
- added C902: ???, Capacitor_THT:CP_Radial_D6.3mm_P2.50mm, F.Cu at (200.8, 55.6)
- added SW201: Reset, Custom:Button 6x3.6mm, F.Cu at (172.8, 81.5)
- added SW202: Boot, Custom:Button 6x3.6mm, F.Cu at (172.8, 77.0)
- moved H111 50.9 mm to (105.6, 95.5)
- moved H112 49.4 mm to (212.4, 48.0)
- moved TP101 45.9 mm to (160.5, 78.6), turned to 0 degrees
- moved J111 30.7 mm to (165.7, 97.7)
- moved TP107 27.1 mm to (142.9, 91.3)
- moved J131 19.1 mm to (210.0, 94.0), turned to 90 degrees
- moved H103 8.93 mm to (211.8, 99.3)
- moved J132 7.96 mm to (210.0, 85.5), turned to 90 degrees
- moved J122 6.90 mm to (189.4, 98.3)
- moved J142 6.90 mm to (189.4, 89.7)
- moved J121 6.90 mm to (182.5, 98.3)
- moved J123 6.90 mm to (196.3, 98.3)
- moved J124 6.90 mm to (203.2, 98.3)
- moved J141 6.90 mm to (182.5, 89.7)
- moved J143 6.90 mm to (196.3, 89.7)
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Connections:
- U201 pad 13: unconnected-(U201-GPIO10-Pad13) -> CAN-L
- U201 pad 14: unconnected-(U201-GPIO11-Pad14) -> CAN-H
- U201 pad 15: unconnected-(U201-GPIO12-Pad15) -> FAN3
- U201 pad 16: unconnected-(U201-GPIO13-Pad16) -> FAN2
- U201 pad 17: unconnected-(U201-GPIO14-Pad17) -> FAN4
- U201 pad 18: unconnected-(U201-GPIO15-Pad18) -> FAN1
- U201 pad 2: unconnected-(U201-GPIO0-Pad2) -> SPI ~{CS} M4
- U201 pad 24: SWCLK -> unconnected-(U201-SWCLK-Pad24)
- U201 pad 25: SWD -> unconnected-(U201-SWD-Pad25)
- U201 pad 28: unconnected-(U201-GPIO17-Pad28) -> RGB
- U201 pad 29: unconnected-(U201-GPIO18-Pad29) -> Bed Heating
- U201 pad 3: unconnected-(U201-GPIO1-Pad3) -> SPI ~{CS} M3
- U201 pad 30: unconnected-(U201-GPIO19-Pad30) -> Head Heating
- U201 pad 34: unconnected-(U201-GPIO22-Pad34) -> Limit 1
- U201 pad 35: unconnected-(U201-GPIO23-Pad35) -> Limit 3
- U201 pad 36: unconnected-(U201-GPIO24-Pad36) -> Limit 2
- U201 pad 37: unconnected-(U201-GPIO25-Pad37) -> Limit 4
- U201 pad 4: unconnected-(U201-GPIO2-Pad4) -> SPI ~{CS} M2
- U201 pad 5: unconnected-(U201-GPIO3-Pad5) -> SPI ~{CS} M1
- U201 pad 6: unconnected-(U201-GPIO4-Pad6) -> SPI MISO
- U201 pad 7: unconnected-(U201-GPIO5-Pad7) -> SPI MOSI
- U201 pad 8: unconnected-(U201-GPIO6-Pad8) -> SPI CLK
- U201 pad 9: unconnected-(U201-GPIO7-Pad9) -> ~{MOTOR ENABLE}
Routing:
- net +48V: track 0.00 -> 90.7 mm, vias 4 -> 6
- net CAN-H: track 12.0 -> 83.8 mm, vias 0 -> 1
- net SPI ~{CS} M4: track 0.00 -> 68.4 mm, vias 0 -> 2
- net CAN-L: track 12.0 -> 77.2 mm, vias 0 -> 1
- net GND: track 121.6 -> 66.8 mm, vias 41 -> 52
- net Head Heating: track 0.00 -> 53.7 mm, vias 0 -> 1
- net SPI MOSI: track 72.0 -> 125.6 mm, vias 0 -> 1
- net SPI CLK: track 72.0 -> 124.8 mm, vias 0 -> 1
- net SPI MISO: track 72.0 -> 124.7 mm, vias 0 -> 1
- net ~{MOTOR ENABLE}: track 72.0 -> 123.4 mm, vias 0 -> 2
- net SPI ~{CS} M3: track 0.00 -> 51.1 mm, vias 0 -> 2
- net Bed Heating: track 0.00 -> 48.9 mm, vias 0 -> 1
- net SPI ~{CS} M1: track 0.00 -> 46.2 mm
- net Limit 4: track 0.00 -> 45.4 mm, vias 0 -> 1
- net Temp 4: track 0.00 -> 44.0 mm
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- added copper zone on B.Cu, net GND
- added copper zone on F.Cu, net GND
- added copper zone on In2.Cu, net GND
- added copper zone on In3.Cu, net GND
Other:
- board text added: "1"
- board text added: "2"
- board text added: "3"
- board text added: "4"
- board text added: "5V GND"
- board text added: "BOOT"
- board text added: "E"
- board text added: "FAN"
- board text added: "GND RGB 5V"
- board text added: "GND Switch 5V"
- board text added: "Heat"
- board text added: "R L"
- board text added: "RESET"
- board text added: "RGB"
- board text added: "Switch"
- board text added: "Temp"
- board text added: "X"
- board text added: "Y"
- board text added: "Z"
- board text removed: "5V RGB GND"
- board text removed: "5V Switch GND"
- board text removed: "GND 5V"
