File: 4MotorCAN.kicad_sch (KiCad schematic)
At the start: 39 parts, among them J101 Molex Micro-Fit 3.0 2x03 - CA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, J102 Molex Micro-Fit 3.0 2x03 - CA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, J111 RGB, J121 Temperature, J122 Temperature, J123 Temperature, J124 Temperature, J131 Heating Enable, J132 Heating Enable, J141 Limit Switch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

Commit message: Finish wiring PCB
Parts:
- J123, J124, J132, J142, J143, J144: now fitted
- TP102, TP103, TP104, TP105, TP106: now not fitted
Other:
- note added: "Crossed TestPoints (DNP) can be measured at LEDs (D101 - D105)"

Commit message: Finish PCB, documentation
Parts:
- D? (x5): now in the parts list
- F102: now left out of the parts list
- R?: value 600 -> 620; LCSC (none) -> C23220
- R?: value 42k -> 47k; LCSC (none) -> C25819; Mouser (none) -> 660-RK73H1JTTD4702F
- R?: value 90k -> 100k; LCSC (none) -> C25803; Mouser (none) -> 667-ERJ-3EKF1003V
- R?: value 18k -> 20k; LCSC (none) -> C4184
Other:
- note added: "18k = 0.5mA"
- note added: "42k = 0.5mA"
- note added: "600 = 0.5mA"
- note added: "90k = 0.5mA"
Changed lines of the file:
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@@
     (stroke (width 0) (type default))
+  )
+  (text "42k = 0.5mA" (at 101.6 48.26 0)
+    (effects (font (size 1.27 1.27)) (justify left bottom))
   )
   (text "Bed Heating" (at 219.71 105.41 0)
@@
   (text "Power LED" (at 91.44 21.59 0)
     (effects (font (size 2.54 2.54)) (justify left bottom))
+  )
+  (text "90k = 0.5mA" (at 101.6 35.56 0)
+    (effects (font (size 1.27 1.27)) (justify left bottom))
+  )
+  (text "600 = 0.5mA" (at 101.6 86.36 0)
+    (effects (font (size 1.27 1.27)) (justify left bottom))
   )
   (text "Crossed TestPoints (DNP) can be measured at LEDs (D101 - D105)"
@@
   (text "Heating enable" (at 203.2 82.55 0)
     (effects (font (size 2.54 2.54)) (justify left bottom))
+  )
+  (text "18k = 0.5mA" (at 101.6 60.96 0)
+    (effects (font (size 1.27 1.27)) (justify left bottom))
   )
   (text "RGB LEDs\n (strip)" (at 252.73 25.4 0)
@@
   )
   (symbol (lib_id "Device:LED") (at 97.79 44.45 0) (mirror x) (unit 1)
-    (in_bom no) (on_board yes) (dnp no)
+    (in_bom yes) (on_board yes) (dnp no)
     (property "Reference" "D?" (at 96.52 40.64 0)
       (effects (font (size 1.27 1.27)))
@@
   )
   (symbol (lib_id "Device:LED") (at 97.79 57.15 0) (mirror x) (unit 1)
-    (in_bom no) (on_board yes) (dnp no)
+    (in_bom yes) (on_board yes) (dnp no)
     (property "Reference" "D?" (at 96.52 53.34 0)
       (effects (font (size 1.27 1.27)))
@@
   )
   (symbol (lib_id "Device:LED") (at 97.79 31.75 0) (mirror x) (unit 1)
-    (in_bom no) (on_board yes) (dnp no)
+    (in_bom yes) (on_board yes) (dnp no)
     (property "Reference" "D?" (at 96.52 27.94 0)
       (effects (font (size 1.27 1.27)))
@@
   )
   (symbol (lib_id "Device:LED") (at 97.79 82.55 0) (mirror x) (unit 1)
-    (in_bom no) (on_board yes) (dnp no)
+    (in_bom yes) (on_board yes) (dnp no)
     (property "Reference" "D?" (at 96.52 78.74 0)
       (effects (font (size 1.27 1.27)))
@@
       (effects (font (size 1.27 1.27)))
     )
-    (property "Value" "600" (at 105.41 82.55 90)
+    (property "Value" "620" (at 105.41 82.55 90)
       (effects (font (size 1.27 1.27)))
     )
@@
       (effects (font (size 1.27 1.27)) hide)
     )
-    (property "LCSC" "" (at 105.41 82.55 0)
+    (property "LCSC" "C23220" (at 105.41 82.55 0)
       (effects (font (size 1.27 1.27)) hide)
     )
@@
       (effects (font (size 1.27 1.27)))
     )
-    (property "Value" "42k" (at 105.41 44.45 90)
+    (property "Value" "47k" (at 105.41 44.45 90)
       (effects (font (size 1.27 1.27)))
     )
@@
       (effects (font (size 1.27 1.27)) hide)
     )
-    (property "LCSC" "" (at 105.41 44.45 0)
-      (effects (font (size 1.27 1.27)) hide)
-    )
-    (property "Mouser" "" (at 105.41 44.45 0)
+    (property "LCSC" "C25819" (at 105.41 44.45 0)
+      (effects (font (size 1.27 1.27)) hide)
+    )
+    (property "Mouser" "660-RK73H1JTTD4702F" (at 105.41 44.45 0)
       (effects (font (size 1.27 1.27)) hide)
     )
@@
       (effects (font (size 1.27 1.27)))
     )
-    (property "Value" "90k" (at 105.41 31.75 90)
+    (property "Value" "100k" (at 105.41 31.75 90)
       (effects (font (size 1.27 1.27)))
     )
@@
       (effects (font (size 1.27 1.27)) hide)
     )
-    (property "LCSC" "" (at 105.41 31.75 0)
-      (effects (font (size 1.27 1.27)) hide)
-    )
-    (property "Mouser" "" (at 105.41 31.75 0)
+    (property "LCSC" "C25803" (at 105.41 31.75 0)
+      (effects (font (size 1.27 1.27)) hide)
+    )
+    (property "Mouser" "667-ERJ-3EKF1003V" (at 105.41 31.75 0)
       (effects (font (size 1.27 1.27)) hide)
     )
@@
       (effects (font (size 1.27 1.27)))
     )
-    (property "Value" "18k" (at 105.41 57.15 90)
+    (property "Value" "20k" (at 105.41 57.15 90)
       (effects (font (size 1.27 1.27)))
     )
@@
       (effects (font (size 1.27 1.27)) hide)
     )
-    (property "LCSC" "" (at 105.41 57.15 0)
+    (property "LCSC" "C4184" (at 105.41 57.15 0)
       (effects (font (size 1.27 1.27)) hide)
     )
@@
   )
   (symbol (lib_id "Device:LED") (at 97.79 69.85 0) (mirror x) (unit 1)
-    (in_bom no) (on_board yes) (dnp no)
+    (in_bom yes) (on_board yes) (dnp no)
     (property "Reference" "D?" (at 96.52 66.04 0)
       (effects (font (size 1.27 1.27)))
@@
   )
   (symbol (lib_id "Device:Polyfuse") (at 58.42 157.48 180) (unit 1)
-    (in_bom yes) (on_board yes) (dnp yes)
+    (in_bom no) (on_board yes) (dnp yes)
     (property "Reference" "F102" (at 57.15 156.21 0)
       (effects (font (size 1.27 1.27)) (justify left))
