File: Motor1.kicad_sch (KiCad schematic)
At the start: 15 parts, among them J603 Direction, U601 FYSETC TMC5160

Commit message: Finish PCB, documentation
Parts:
- C? (x2), J603, R? (x5): now left out of the parts list
- D?: now in the parts list
Changed lines of the file:
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@@
   )
   (symbol (lib_id "Device:R_Small") (at 95.25 173.99 90) (unit 1)
-    (in_bom yes) (on_board yes) (dnp yes)
+    (in_bom no) (on_board yes) (dnp yes)
     (property "Reference" "R?" (at 95.25 171.45 90)
       (effects (font (size 1.27 1.27)))
@@
   )
   (symbol (lib_id "Device:C_Small") (at 91.44 176.53 0) (mirror y) (unit 1)
-    (in_bom yes) (on_board yes) (dnp yes)
+    (in_bom no) (on_board yes) (dnp yes)
     (property "Reference" "C?" (at 88.9 175.2663 0)
       (effects (font (size 1.27 1.27)) (justify left))
@@
   )
   (symbol (lib_id "Device:R_Small") (at 100.33 171.45 0) (mirror x) (unit 1)
-    (in_bom yes) (on_board yes) (dnp yes)
+    (in_bom no) (on_board yes) (dnp yes)
     (property "Reference" "R?" (at 101.6 170.18 0)
       (effects (font (size 1.27 1.27)) (justify left))
@@
   )
   (symbol (lib_id "Device:C_Small") (at 130.81 176.53 0) (unit 1)
-    (in_bom yes) (on_board yes) (dnp yes)
+    (in_bom no) (on_board yes) (dnp yes)
     (property "Reference" "C?" (at 133.35 175.2663 0)
       (effects (font (size 1.27 1.27)) (justify left))
@@
   )
   (symbol (lib_id "Device:R_Small") (at 43.18 163.83 90) (unit 1)
-    (in_bom yes) (on_board yes) (dnp yes)
+    (in_bom no) (on_board yes) (dnp yes)
     (property "Reference" "R?" (at 43.18 161.29 90)
       (effects (font (size 1.27 1.27)))
@@
   )
   (symbol (lib_id "Connector_Generic:Conn_02x02_Odd_Even") (at 110.49 180.34 0) (mirror x) (unit 1)
-    (in_bom yes) (on_board yes) (dnp yes)
+    (in_bom no) (on_board yes) (dnp yes)
     (property "Reference" "J603" (at 111.76 175.26 0)
       (effects (font (size 1.27 1.27)))
@@
   )
   (symbol (lib_id "Device:LED") (at 39.37 173.99 0) (mirror x) (unit 1)
-    (in_bom no) (on_board yes) (dnp no)
+    (in_bom yes) (on_board yes) (dnp no)
     (property "Reference" "D?" (at 38.1 170.18 0)
       (effects (font (size 1.27 1.27)))
@@
   )
   (symbol (lib_id "Device:R_Small") (at 127 173.99 270) (mirror x) (unit 1)
-    (in_bom yes) (on_board yes) (dnp yes)
+    (in_bom no) (on_board yes) (dnp yes)
     (property "Reference" "R?" (at 127 171.45 90)
       (effects (font (size 1.27 1.27)))
@@
   )
   (symbol (lib_id "Device:R_Small") (at 121.92 171.45 180) (unit 1)
-    (in_bom yes) (on_board yes) (dnp yes)
+    (in_bom no) (on_board yes) (dnp yes)
     (property "Reference" "R?" (at 120.65 170.18 0)
       (effects (font (size 1.27 1.27)) (justify left))
